Commit message: YA TIENE EL SCARA

File: PRACTICA1-URDF/modelo.urdf (robot description, URDF)
Before this commit: robot spherical_robot, 4 links, 3 joints
Links:
- removed link arm_link
- removed link forearm_link
- removed link shoulder_link
- added link arm_1; visual box size=0.5 0.05 0.05
- added link arm_2; visual box size=0.50 0.05 0.05
- added link end_effector; visual cylinder length=0.1 radius=0.02
- added link vertical_axis; visual cylinder length=0.15 radius=0.03
- link base_link: geometry visual cylinder length=0.2 radius=0.1
Joints:
- removed joint arm_joint
- removed joint forearm_joint
- removed joint shoulder_joint
- added joint joint_1: type revolute, parent base_link, child arm_1, origin xyz=0 0 0.1 rpy=0 0 0, axis 0 0 1, limit lower=-1.57 upper=1.57 effort=50 velocity=1.5
- added joint joint_2: type revolute, parent arm_1, child arm_2, origin xyz=0.2 0 0 rpy=0 0 0, axis 0 0 1, limit lower=-1.57 upper=1.57 effort=50 velocity=1.5
- added joint joint_3: type prismatic, parent arm_2, child vertical_axis, origin xyz=0.25 0 0 rpy=0 0 0, axis 0 0 -1, limit lower=-0.1 upper=0 effort=30 velocity=0.5
- added joint joint_4: type revolute, parent vertical_axis, child end_effector, origin xyz=0 0 -0.1 rpy=0 0 0, axis 0 0 1, limit lower=-3.14 upper=3.14 effort=10 velocity=2.0

Commit message: MODIFICADO 20.03.25

File: PRACTICA1-URDF/modelo.urdf (robot description, URDF)
Before this commit: robot scara_robot, 5 links, 4 joints
Links:
- link base_link: geometry visual cylinder length=0.4 radius=0.1
- link end_effector: geometry visual cylinder length=0.14 radius=0.02
Joints:
- joint joint_1: limit lower=-1.57 upper=1.57 effort=50 velocity=1.5 -> lower=-3.14 upper=3.14 effort=50 velocity=1.5; origin xyz=0 0 0.1 rpy=0 0 0 -> xyz=0 0 0.4 rpy=0 0 0
- joint joint_2: limit lower=-1.57 upper=1.57 effort=50 velocity=1.5 -> lower=-2.5 upper=2.5 effort=50 velocity=1.5; origin xyz=0.2 0 0 rpy=0 0 0 -> xyz=0.23 0 0 rpy=0 0 0
- joint joint_3: axis 0 0 -1 -> (none); limit lower=-0.1 upper=0 effort=30 velocity=0.5 -> (none); type prismatic -> fixed
- joint joint_4: axis 0 0 1 -> 0 0 -1; limit lower=-3.14 upper=3.14 effort=10 velocity=2.0 -> lower=-0.1 upper=0 effort=30 velocity=0.5; type revolute -> prismatic
